Commit message: 1.4.5 Modify some maximum joint effort values

File: tm_description/xacro/macro.tm12s-nominal.urdf.xacro (robot description, xacro)
@@ -15,10 +15,10 @@
     joint_5_velocity_limit:=${radians(225)}
     joint_6_velocity_limit:=${radians(450)}
-    joint_1_effort_limit:=${350}
-    joint_2_effort_limit:=${350}
-    joint_3_effort_limit:=${170}
-    joint_4_effort_limit:=${45}
-    joint_5_effort_limit:=${45}
-    joint_6_effort_limit:=${45}
+    joint_1_effort_limit:=${353}
+    joint_2_effort_limit:=${353}
+    joint_3_effort_limit:=${157}
+    joint_4_effort_limit:=${54}
+    joint_5_effort_limit:=${54}
+    joint_6_effort_limit:=${34}
     safety_limits:=false safety_pos_margin:=0.15
     safety_k_position:=20">

File: tm_description/xacro/macro.tm12sx-nominal.urdf.xacro (robot description, xacro)
@@ -15,10 +15,10 @@
     joint_5_velocity_limit:=${radians(225)}
     joint_6_velocity_limit:=${radians(450)}
-    joint_1_effort_limit:=${350}
-    joint_2_effort_limit:=${350}
-    joint_3_effort_limit:=${170}
-    joint_4_effort_limit:=${45}
-    joint_5_effort_limit:=${45}
-    joint_6_effort_limit:=${45}
+    joint_1_effort_limit:=${353}
+    joint_2_effort_limit:=${353}
+    joint_3_effort_limit:=${157}
+    joint_4_effort_limit:=${54}
+    joint_5_effort_limit:=${54}
+    joint_6_effort_limit:=${34}
     safety_limits:=false safety_pos_margin:=0.15
     safety_k_position:=20">
@@ -88,5 +88,5 @@
       </xacro:if>
       <xacro:if value="${prefix_monochrome_command}">
-      <material name="${color}" />
+        <material name="${color}" />
       </xacro:if>
     </visual>
@@ -122,5 +122,5 @@
       </xacro:if>
       <xacro:if value="${prefix_monochrome_command}">
-      <material name="${color}" />
+        <material name="${color}" />
       </xacro:if>
     </visual>
@@ -157,5 +157,5 @@
       </xacro:if>
       <xacro:if value="${prefix_monochrome_command}">
-      <material name="${color}" />
+        <material name="${color}" />
       </xacro:if>
     </visual>
@@ -192,5 +192,5 @@
       </xacro:if>
       <xacro:if value="${prefix_monochrome_command}">
-      <material name="${color}" />
+        <material name="${color}" />
       </xacro:if>
     </visual>
@@ -227,5 +227,5 @@
       </xacro:if>
       <xacro:if value="${prefix_monochrome_command}">
-      <material name="${color}" />
+        <material name="${color}" />
       </xacro:if>
     </visual>
@@ -262,5 +262,5 @@
       </xacro:if>
       <xacro:if value="${prefix_monochrome_command}">
-      <material name="${color}" />
+        <material name="${color}" />
       </xacro:if>
     </visual>
@@ -297,5 +297,5 @@
       </xacro:if>
       <xacro:if value="${prefix_monochrome_command}">
-      <material name="${color}" />
+        <material name="${color}" />
       </xacro:if>
     </visual>

File: tm_description/xacro/macro.tm14s-nominal.urdf.xacro (robot description, xacro)
@@ -15,10 +15,10 @@
     joint_5_velocity_limit:=${radians(225)}
     joint_6_velocity_limit:=${radians(450)}
-    joint_1_effort_limit:=${350}
-    joint_2_effort_limit:=${350}
-    joint_3_effort_limit:=${170}
-    joint_4_effort_limit:=${45}
-    joint_5_effort_limit:=${45}
-    joint_6_effort_limit:=${45}
+    joint_1_effort_limit:=${353}
+    joint_2_effort_limit:=${353}
+    joint_3_effort_limit:=${157}
+    joint_4_effort_limit:=${54}
+    joint_5_effort_limit:=${54}
+    joint_6_effort_limit:=${34}
     safety_limits:=false safety_pos_margin:=0.15
     safety_k_position:=20">
@@ -88,5 +88,5 @@
       </xacro:if>
       <xacro:if value="${prefix_monochrome_command}">
-      <material name="${color}" />
+        <material name="${color}" />
       </xacro:if>
     </visual>
@@ -122,5 +122,5 @@
       </xacro:if>
       <xacro:if value="${prefix_monochrome_command}">
-      <material name="${color}" />
+        <material name="${color}" />
       </xacro:if>
     </visual>
@@ -157,5 +157,5 @@
       </xacro:if>
       <xacro:if value="${prefix_monochrome_command}">
-      <material name="${color}" />
+        <material name="${color}" />
       </xacro:if>
     </visual>
@@ -192,5 +192,5 @@
       </xacro:if>
       <xacro:if value="${prefix_monochrome_command}">
-      <material name="${color}" />
+        <material name="${color}" />
       </xacro:if>
     </visual>
@@ -227,5 +227,5 @@
       </xacro:if>
       <xacro:if value="${prefix_monochrome_command}">
-      <material name="${color}" />
+        <material name="${color}" />
       </xacro:if>
     </visual>
@@ -262,5 +262,5 @@
       </xacro:if>
       <xacro:if value="${prefix_monochrome_command}">
-      <material name="${color}" />
+        <material name="${color}" />
       </xacro:if>
     </visual>
@@ -297,5 +297,5 @@
       </xacro:if>
       <xacro:if value="${prefix_monochrome_command}">
-      <material name="${color}" />
+        <material name="${color}" />
       </xacro:if>
     </visual>

File: tm_description/xacro/macro.tm14sx-nominal.urdf.xacro (robot description, xacro)
@@ -15,10 +15,10 @@
     joint_5_velocity_limit:=${radians(225)}
     joint_6_velocity_limit:=${radians(450)}
-    joint_1_effort_limit:=${350}
-    joint_2_effort_limit:=${350}
-    joint_3_effort_limit:=${170}
-    joint_4_effort_limit:=${45}
-    joint_5_effort_limit:=${45}
-    joint_6_effort_limit:=${45}
+    joint_1_effort_limit:=${353}
+    joint_2_effort_limit:=${353}
+    joint_3_effort_limit:=${157}
+    joint_4_effort_limit:=${54}
+    joint_5_effort_limit:=${54}
+    joint_6_effort_limit:=${34}
     safety_limits:=false safety_pos_margin:=0.15
     safety_k_position:=20">
@@ -88,5 +88,5 @@
       </xacro:if>
       <xacro:if value="${prefix_monochrome_command}">
-      <material name="${color}" />
+        <material name="${color}" />
       </xacro:if>
     </visual>
@@ -122,5 +122,5 @@
       </xacro:if>
       <xacro:if value="${prefix_monochrome_command}">
-      <material name="${color}" />
+        <material name="${color}" />
       </xacro:if>
     </visual>
@@ -157,5 +157,5 @@
       </xacro:if>
       <xacro:if value="${prefix_monochrome_command}">
-      <material name="${color}" />
+        <material name="${color}" />
       </xacro:if>
     </visual>
@@ -192,5 +192,5 @@
       </xacro:if>
       <xacro:if value="${prefix_monochrome_command}">
-      <material name="${color}" />
+        <material name="${color}" />
       </xacro:if>
     </visual>
@@ -227,5 +227,5 @@
       </xacro:if>
       <xacro:if value="${prefix_monochrome_command}">
-      <material name="${color}" />
+        <material name="${color}" />
       </xacro:if>
     </visual>
@@ -262,5 +262,5 @@
       </xacro:if>
       <xacro:if value="${prefix_monochrome_command}">
-      <material name="${color}" />
+        <material name="${color}" />
       </xacro:if>
     </visual>
@@ -297,5 +297,5 @@
       </xacro:if>
       <xacro:if value="${prefix_monochrome_command}">
-      <material name="${color}" />
+        <material name="${color}" />
       </xacro:if>
     </visual>

File: tm_description/xacro/macro.tm25s-nominal.urdf.xacro (robot description, xacro)
@@ -88,5 +88,5 @@
       </xacro:if>
       <xacro:if value="${prefix_monochrome_command}">
-      <material name="${color}" />
+        <material name="${color}" />
       </xacro:if>
     </visual>
@@ -122,5 +122,5 @@
       </xacro:if>
       <xacro:if value="${prefix_monochrome_command}">
-      <material name="${color}" />
+        <material name="${color}" />
       </xacro:if>
     </visual>
@@ -157,5 +157,5 @@
       </xacro:if>
       <xacro:if value="${prefix_monochrome_command}">
-      <material name="${color}" />
+        <material name="${color}" />
       </xacro:if>
     </visual>
@@ -192,5 +192,5 @@
       </xacro:if>
       <xacro:if value="${prefix_monochrome_command}">
-      <material name="${color}" />
+        <material name="${color}" />
       </xacro:if>
     </visual>
@@ -227,5 +227,5 @@
       </xacro:if>
       <xacro:if value="${prefix_monochrome_command}">
-      <material name="${color}" />
+        <material name="${color}" />
       </xacro:if>
     </visual>
@@ -262,5 +262,5 @@
       </xacro:if>
       <xacro:if value="${prefix_monochrome_command}">
-      <material name="${color}" />
+        <material name="${color}" />
       </xacro:if>
     </visual>
@@ -297,5 +297,5 @@
       </xacro:if>
       <xacro:if value="${prefix_monochrome_command}">
-      <material name="${color}" />
+        <material name="${color}" />
       </xacro:if>
     </visual>

File: tm_description/xacro/macro.tm25sx-nominal.urdf.xacro (robot description, xacro)
@@ -88,5 +88,5 @@
       </xacro:if>
       <xacro:if value="${prefix_monochrome_command}">
-      <material name="${color}" />
+        <material name="${color}" />
       </xacro:if>
     </visual>
@@ -122,5 +122,5 @@
       </xacro:if>
       <xacro:if value="${prefix_monochrome_command}">
-      <material name="${color}" />
+        <material name="${color}" />
       </xacro:if>
     </visual>
@@ -157,5 +157,5 @@
       </xacro:if>
       <xacro:if value="${prefix_monochrome_command}">
-      <material name="${color}" />
+        <material name="${color}" />
       </xacro:if>
     </visual>
@@ -192,5 +192,5 @@
       </xacro:if>
       <xacro:if value="${prefix_monochrome_command}">
-      <material name="${color}" />
+        <material name="${color}" />
       </xacro:if>
     </visual>
@@ -227,5 +227,5 @@
       </xacro:if>
       <xacro:if value="${prefix_monochrome_command}">
-      <material name="${color}" />
+        <material name="${color}" />
       </xacro:if>
     </visual>
@@ -262,5 +262,5 @@
       </xacro:if>
       <xacro:if value="${prefix_monochrome_command}">
-      <material name="${color}" />
+        <material name="${color}" />
       </xacro:if>
     </visual>
@@ -297,5 +297,5 @@
       </xacro:if>
       <xacro:if value="${prefix_monochrome_command}">
-      <material name="${color}" />
+        <material name="${color}" />
       </xacro:if>
     </visual>

File: tm_description/xacro/macro.tm30s-nominal.urdf.xacro (robot description, xacro)
@@ -88,5 +88,5 @@
       </xacro:if>
       <xacro:if value="${prefix_monochrome_command}">
-      <material name="${color}" />
+        <material name="${color}" />
       </xacro:if>
     </visual>
@@ -122,5 +122,5 @@
       </xacro:if>
       <xacro:if value="${prefix_monochrome_command}">
-      <material name="${color}" />
+        <material name="${color}" />
       </xacro:if>
     </visual>
@@ -157,5 +157,5 @@
       </xacro:if>
       <xacro:if value="${prefix_monochrome_command}">
-      <material name="${color}" />
+        <material name="${color}" />
       </xacro:if>
     </visual>
@@ -192,5 +192,5 @@
       </xacro:if>
       <xacro:if value="${prefix_monochrome_command}">
-      <material name="${color}" />
+        <material name="${color}" />
       </xacro:if>
     </visual>
@@ -227,5 +227,5 @@
       </xacro:if>
       <xacro:if value="${prefix_monochrome_command}">
-      <material name="${color}" />
+        <material name="${color}" />
       </xacro:if>
     </visual>
@@ -262,5 +262,5 @@
       </xacro:if>
       <xacro:if value="${prefix_monochrome_command}">
-      <material name="${color}" />
+        <material name="${color}" />
       </xacro:if>
     </visual>
@@ -297,5 +297,5 @@
       </xacro:if>
       <xacro:if value="${prefix_monochrome_command}">
-      <material name="${color}" />
+        <material name="${color}" />
       </xacro:if>
     </visual>

File: tm_description/xacro/macro.tm30sx-nominal.urdf.xacro (robot description, xacro)
@@ -88,5 +88,5 @@
       </xacro:if>
       <xacro:if value="${prefix_monochrome_command}">
-      <material name="${color}" />
+        <material name="${color}" />
       </xacro:if>
     </visual>
@@ -122,5 +122,5 @@
       </xacro:if>
       <xacro:if value="${prefix_monochrome_command}">
-      <material name="${color}" />
+        <material name="${color}" />
       </xacro:if>
     </visual>
@@ -157,5 +157,5 @@
       </xacro:if>
       <xacro:if value="${prefix_monochrome_command}">
-      <material name="${color}" />
+        <material name="${color}" />
       </xacro:if>
     </visual>
@@ -192,5 +192,5 @@
       </xacro:if>
       <xacro:if value="${prefix_monochrome_command}">
-      <material name="${color}" />
+        <material name="${color}" />
       </xacro:if>
     </visual>
@@ -227,5 +227,5 @@
       </xacro:if>
       <xacro:if value="${prefix_monochrome_command}">
-      <material name="${color}" />
+        <material name="${color}" />
       </xacro:if>
     </visual>
@@ -262,5 +262,5 @@
       </xacro:if>
       <xacro:if value="${prefix_monochrome_command}">
-      <material name="${color}" />
+        <material name="${color}" />
       </xacro:if>
     </visual>
@@ -297,5 +297,5 @@
       </xacro:if>
       <xacro:if value="${prefix_monochrome_command}">
-      <material name="${color}" />
+        <material name="${color}" />
       </xacro:if>
     </visual>

File: tm_description/xacro/macro.tm5s-nominal.urdf.xacro (robot description, xacro)
@@ -15,10 +15,10 @@
     joint_5_velocity_limit:=${radians(225)}
     joint_6_velocity_limit:=${radians(450)}
-    joint_1_effort_limit:=${170}
-    joint_2_effort_limit:=${170}
-    joint_3_effort_limit:=${170}
-    joint_4_effort_limit:=${45}
-    joint_5_effort_limit:=${45}
-    joint_6_effort_limit:=${45}
+    joint_1_effort_limit:=${157}
+    joint_2_effort_limit:=${157}
+    joint_3_effort_limit:=${157}
+    joint_4_effort_limit:=${54}
+    joint_5_effort_limit:=${54}
+    joint_6_effort_limit:=${34}
     safety_limits:=false safety_pos_margin:=0.15
     safety_k_position:=20">
@@ -88,5 +88,5 @@
       </xacro:if>
       <xacro:if value="${prefix_monochrome_command}">
-      <material name="${color}" />
+        <material name="${color}" />
       </xacro:if>
     </visual>
@@ -122,5 +122,5 @@
       </xacro:if>
       <xacro:if value="${prefix_monochrome_command}">
-      <material name="${color}" />
+        <material name="${color}" />
       </xacro:if>
     </visual>
@@ -157,5 +157,5 @@
       </xacro:if>
       <xacro:if value="${prefix_monochrome_command}">
-      <material name="${color}" />
+        <material name="${color}" />
       </xacro:if>
     </visual>
@@ -192,5 +192,5 @@
       </xacro:if>
       <xacro:if value="${prefix_monochrome_command}">
-      <material name="${color}" />
+        <material name="${color}" />
       </xacro:if>
     </visual>
@@ -227,5 +227,5 @@
       </xacro:if>
       <xacro:if value="${prefix_monochrome_command}">
-      <material name="${color}" />
+        <material name="${color}" />
       </xacro:if>
     </visual>
@@ -262,5 +262,5 @@
       </xacro:if>
       <xacro:if value="${prefix_monochrome_command}">
-      <material name="${color}" />
+        <material name="${color}" />
       </xacro:if>
     </visual>
@@ -297,5 +297,5 @@
       </xacro:if>
       <xacro:if value="${prefix_monochrome_command}">
-      <material name="${color}" />
+        <material name="${color}" />
       </xacro:if>
     </visual>

File: tm_description/xacro/macro.tm5sx-nominal.urdf.xacro (robot description, xacro)
@@ -15,10 +15,10 @@
     joint_5_velocity_limit:=${radians(225)}
     joint_6_velocity_limit:=${radians(450)}
-    joint_1_effort_limit:=${170}
-    joint_2_effort_limit:=${170}
-    joint_3_effort_limit:=${170}
-    joint_4_effort_limit:=${45}
-    joint_5_effort_limit:=${45}
-    joint_6_effort_limit:=${45}
+    joint_1_effort_limit:=${157}
+    joint_2_effort_limit:=${157}
+    joint_3_effort_limit:=${157}
+    joint_4_effort_limit:=${54}
+    joint_5_effort_limit:=${54}
+    joint_6_effort_limit:=${34}
     safety_limits:=false safety_pos_margin:=0.15
     safety_k_position:=20">
@@ -88,5 +88,5 @@
       </xacro:if>
       <xacro:if value="${prefix_monochrome_command}">
-      <material name="${color}" />
+        <material name="${color}" />
       </xacro:if>
     </visual>
@@ -122,5 +122,5 @@
       </xacro:if>
       <xacro:if value="${prefix_monochrome_command}">
-      <material name="${color}" />
+        <material name="${color}" />
       </xacro:if>
     </visual>
@@ -157,5 +157,5 @@
       </xacro:if>
       <xacro:if value="${prefix_monochrome_command}">
-      <material name="${color}" />
+        <material name="${color}" />
       </xacro:if>
     </visual>
@@ -192,5 +192,5 @@
       </xacro:if>
       <xacro:if value="${prefix_monochrome_command}">
-      <material name="${color}" />
+        <material name="${color}" />
       </xacro:if>
     </visual>
@@ -227,5 +227,5 @@
       </xacro:if>
       <xacro:if value="${prefix_monochrome_command}">
-      <material name="${color}" />
+        <material name="${color}" />
       </xacro:if>
     </visual>
@@ -262,5 +262,5 @@
       </xacro:if>
       <xacro:if value="${prefix_monochrome_command}">
-      <material name="${color}" />
+        <material name="${color}" />
       </xacro:if>
     </visual>
@@ -297,5 +297,5 @@
       </xacro:if>
       <xacro:if value="${prefix_monochrome_command}">
-      <material name="${color}" />
+        <material name="${color}" />
       </xacro:if>
     </visual>

File: tm_description/xacro/macro.tm7s-nominal.urdf.xacro (robot description, xacro)
@@ -15,10 +15,10 @@
     joint_5_velocity_limit:=${radians(225)}
     joint_6_velocity_limit:=${radians(450)}
-    joint_1_effort_limit:=${170}
-    joint_2_effort_limit:=${170}
-    joint_3_effort_limit:=${170}
-    joint_4_effort_limit:=${45}
-    joint_5_effort_limit:=${45}
-    joint_6_effort_limit:=${45}
+    joint_1_effort_limit:=${157}
+    joint_2_effort_limit:=${157}
+    joint_3_effort_limit:=${157}
+    joint_4_effort_limit:=${54}
+    joint_5_effort_limit:=${54}
+    joint_6_effort_limit:=${34}
     safety_limits:=false safety_pos_margin:=0.15
     safety_k_position:=20">
@@ -88,5 +88,5 @@
       </xacro:if>
       <xacro:if value="${prefix_monochrome_command}">
-      <material name="${color}" />
+        <material name="${color}" />
       </xacro:if>
     </visual>
@@ -122,5 +122,5 @@
       </xacro:if>
       <xacro:if value="${prefix_monochrome_command}">
-      <material name="${color}" />
+        <material name="${color}" />
       </xacro:if>
     </visual>
@@ -157,5 +157,5 @@
       </xacro:if>
       <xacro:if value="${prefix_monochrome_command}">
-      <material name="${color}" />
+        <material name="${color}" />
       </xacro:if>
     </visual>
@@ -192,5 +192,5 @@
       </xacro:if>
       <xacro:if value="${prefix_monochrome_command}">
-      <material name="${color}" />
+        <material name="${color}" />
       </xacro:if>
     </visual>
@@ -227,5 +227,5 @@
       </xacro:if>
       <xacro:if value="${prefix_monochrome_command}">
-      <material name="${color}" />
+        <material name="${color}" />
       </xacro:if>
     </visual>
@@ -262,5 +262,5 @@
       </xacro:if>
       <xacro:if value="${prefix_monochrome_command}">
-      <material name="${color}" />
+        <material name="${color}" />
       </xacro:if>
     </visual>
@@ -297,5 +297,5 @@
       </xacro:if>
       <xacro:if value="${prefix_monochrome_command}">
-      <material name="${color}" />
+        <material name="${color}" />
       </xacro:if>
     </visual>

File: tm_description/xacro/macro.tm7sx-nominal.urdf.xacro (robot description, xacro)
@@ -15,10 +15,10 @@
     joint_5_velocity_limit:=${radians(225)}
     joint_6_velocity_limit:=${radians(450)}
-    joint_1_effort_limit:=${170}
-    joint_2_effort_limit:=${170}
-    joint_3_effort_limit:=${170}
-    joint_4_effort_limit:=${45}
-    joint_5_effort_limit:=${45}
-    joint_6_effort_limit:=${45}
+    joint_1_effort_limit:=${157}
+    joint_2_effort_limit:=${157}
+    joint_3_effort_limit:=${157}
+    joint_4_effort_limit:=${54}
+    joint_5_effort_limit:=${54}
+    joint_6_effort_limit:=${34}
     safety_limits:=false safety_pos_margin:=0.15
     safety_k_position:=20">
@@ -88,5 +88,5 @@
       </xacro:if>
       <xacro:if value="${prefix_monochrome_command}">
-      <material name="${color}" />
+        <material name="${color}" />
       </xacro:if>
     </visual>
@@ -122,5 +122,5 @@
       </xacro:if>
       <xacro:if value="${prefix_monochrome_command}">
-      <material name="${color}" />
+        <material name="${color}" />
       </xacro:if>
     </visual>
@@ -157,5 +157,5 @@
       </xacro:if>
       <xacro:if value="${prefix_monochrome_command}">
-      <material name="${color}" />
+        <material name="${color}" />
       </xacro:if>
     </visual>
@@ -192,5 +192,5 @@
       </xacro:if>
       <xacro:if value="${prefix_monochrome_command}">
-      <material name="${color}" />
+        <material name="${color}" />
       </xacro:if>
     </visual>
@@ -227,5 +227,5 @@
       </xacro:if>
       <xacro:if value="${prefix_monochrome_command}">
-      <material name="${color}" />
+        <material name="${color}" />
       </xacro:if>
     </visual>
@@ -262,5 +262,5 @@
       </xacro:if>
       <xacro:if value="${prefix_monochrome_command}">
-      <material name="${color}" />
+        <material name="${color}" />
       </xacro:if>
     </visual>
@@ -297,5 +297,5 @@
       </xacro:if>
       <xacro:if value="${prefix_monochrome_command}">
-      <material name="${color}" />
+        <material name="${color}" />
       </xacro:if>
     </visual>

File: tm_gazebo/xacro/macro.tm12s-nominal.urdf.xacro (robot description, xacro)
@@ -15,10 +15,10 @@
     joint_5_velocity_limit:=${radians(225)}
     joint_6_velocity_limit:=${radians(450)}
-    joint_1_effort_limit:=${350}
-    joint_2_effort_limit:=${350}
-    joint_3_effort_limit:=${170}
-    joint_4_effort_limit:=${45}
-    joint_5_effort_limit:=${45}
-    joint_6_effort_limit:=${45}
+    joint_1_effort_limit:=${353}
+    joint_2_effort_limit:=${353}
+    joint_3_effort_limit:=${157}
+    joint_4_effort_limit:=${54}
+    joint_5_effort_limit:=${54}
+    joint_6_effort_limit:=${34}
     safety_limits:=false safety_pos_margin:=0.15
     safety_k_position:=20">

File: tm_gazebo/xacro/macro.tm12sx-nominal.urdf.xacro (robot description, xacro)
@@ -15,10 +15,10 @@
     joint_5_velocity_limit:=${radians(225)}
     joint_6_velocity_limit:=${radians(450)}
-    joint_1_effort_limit:=${350}
-    joint_2_effort_limit:=${350}
-    joint_3_effort_limit:=${170}
-    joint_4_effort_limit:=${45}
-    joint_5_effort_limit:=${45}
-    joint_6_effort_limit:=${45}
+    joint_1_effort_limit:=${353}
+    joint_2_effort_limit:=${353}
+    joint_3_effort_limit:=${157}
+    joint_4_effort_limit:=${54}
+    joint_5_effort_limit:=${54}
+    joint_6_effort_limit:=${34}
     safety_limits:=false safety_pos_margin:=0.15
     safety_k_position:=20">
