Commit message: 1.1.6 Modify unit_factor2 value to 1e-6.

File: tm_description/cobot/tm5_900_description/xacro/macro.tm5-900-nominal.urdf.xacro (robot description, xacro)
@@ -64,5 +64,5 @@
     <xacro:property name="izz_5" value="${2643.21*unit_factor}" />
     <xacro:property name="izz_6" value="${1559.496*unit_factor}" />
-    <xacro:property name="unit_factor2" value="0.001"/>
+    <xacro:property name="unit_factor2" value="0.000001"/>
     <xacro:property name="cogx_1" value="${  0.0000000*unit_factor2}" />
     <xacro:property name="cogy_1" value="${  0.0000000*unit_factor2}" />

File: tm_description/cobot_s/tm12s_description/xacro/macro.tm12s-nominal.urdf.xacro (robot description, xacro)
@@ -64,5 +64,5 @@
     <xacro:property name="izz_5" value="${3478.9518*unit_factor}" />
     <xacro:property name="izz_6" value="${1854.4783*unit_factor}" />
-    <xacro:property name="unit_factor2" value="0.001"/>
+    <xacro:property name="unit_factor2" value="0.000001"/>
     <xacro:property name="cogx_1" value="${ -1.0522458*unit_factor2}" />
     <xacro:property name="cogy_1" value="${ -5411.0119*unit_factor2}" />
